File: TCA9548A/TCA9548A.sch (KiCad schematic (older format))
At the start: 15 parts, among them J1 Conn_01x12, J2 Conn_01x12, U1 TCA9548APWR

Commit message: Part Numbers Added
Parts:
- C1: Part (none) -> C95841
- R1, R2, R3, R4, R5, R6: Part (none) -> C99198
- U1: Part (none) -> C130026
Changed lines of the file:
@@
 F 2 "Capacitor_SMD:C_0805_2012Metric" H 4113 1800 50  0001 C CNN
 F 3 "~" H 4075 1950 50  0001 C CNN
+F 4 "C95841" H 4075 1950 50  0001 C CNN "Part"
 	1    4075 1950
 	1    0    0    -1
@@
 F 2 "Resistor_SMD:R_0603_1608Metric" V 1515 2665 50  0001 C CNN
 F 3 "~" H 1475 2675 50  0001 C CNN
+F 4 "C99198" H 1475 2675 50  0001 C CNN "Part"
 	1    1475 2675
 	-1   0    0    -1
@@
 F 2 "Package_SO:TSSOP-24_4.4x7.8mm_P0.65mm" H 3025 975 50  0001 C CNN
 F 3 "http://www.ti.com/lit/ds/symlink/tca9548a.pdf" H 3075 2225 50  0001 C CNN
+F 4 "C130026" H 3025 1975 50  0001 C CNN "Part"
 	1    3025 1975
 	1    0    0    -1
@@
 F 2 "Resistor_SMD:R_0603_1608Metric" V 1790 2665 50  0001 C CNN
 F 3 "~" H 1750 2675 50  0001 C CNN
+F 4 "C99198" H 1750 2675 50  0001 C CNN "Part"
 	1    1750 2675
 	-1   0    0    -1
@@
 F 2 "Resistor_SMD:R_0603_1608Metric" V 2065 2665 50  0001 C CNN
 F 3 "~" H 2025 2675 50  0001 C CNN
+F 4 "C99198" H 2025 2675 50  0001 C CNN "Part"
 	1    2025 2675
 	-1   0    0    -1
@@
 F 2 "Resistor_SMD:R_0603_1608Metric" V 2365 1765 50  0001 C CNN
 F 3 "~" H 2325 1775 50  0001 C CNN
+F 4 "C99198" V 2325 1775 50  0001 C CNN "Part"
 	1    2325 1775
 	0    -1   1    0
@@
 F 2 "Resistor_SMD:R_0603_1608Metric" V 1765 1215 50  0001 C CNN
 F 3 "~" H 1725 1225 50  0001 C CNN
+F 4 "C99198" V 1725 1225 50  0001 C CNN "Part"
 	1    1725 1225
 	0    -1   1    0
@@
 F 2 "Resistor_SMD:R_0603_1608Metric" V 1765 1415 50  0001 C CNN
 F 3 "~" H 1725 1425 50  0001 C CNN
+F 4 "C99198" V 1725 1425 50  0001 C CNN "Part"
 	1    1725 1425
 	0    -1   1    0
