File: TCA9548A/TCA9548A.kicad_pcb (KiCad board)
At the start: 2 copper layers, 30.5 x 15.2 mm, 20 parts, among them J1 Conn_01x12, J2 Conn_01x12

Commit message: Minor Updates
Other:
- board text removed: "JLCJLCJLCJLC JLCJLCJLCJLC"
Changed lines of the file:
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@@
   (general
     (thickness 1.6)
-    (drawings 40)
+    (drawings 39)
     (tracks 166)
     (zones 0)
@@
   )
   (setup
-    (last_trace_width 0.5)
+    (last_trace_width 0.127)
     (user_trace_width 0.127)
     (user_trace_width 0.15)
@@
     (effects (font (size 0.9 0.8) (thickness 0.13)))
   )
-  (gr_text "JLCJLCJLCJLC\nJLCJLCJLCJLC" (at 66.04 35.306 90) (layer F.SilkS)
-    (effects (font (size 0.9 0.8) (thickness 0.13)))
-  )
